File: esp.kicad_sch (KiCad schematic)
At the start: 12 parts, among them J3 DEBUG, J6 EXTRA, SW1 SW, SW2 SW, U1 ESP32-WROOM-32

Commit message: Routing almost finished
Parts:
- added D3, D4: LED, LED_SMD:LED_0603_1608Metric, symbol Device:LED
- added R48, R49: 330, Resistor_SMD:R_0603_1608Metric, symbol rflib:R
- added R51, R52: 10k, Resistor_SMD:R_0603_1608Metric, symbol rflib:R
- J6: footprint Connector_PinHeader_1.00mm:PinHeader_1x05_P1.00mm_Vertical -> Connector_PinHeader_2.54mm:PinHeader_1x05_P2.54mm_Vertical
Connections:
- net GND: now also D3.1 (K), D4.1 (K)
- net LED_A: now reaches U1.14 (IO12)
- net LED_A: now also R52.1
- net LED_B: now reaches U1.16 (IO13)
- net LED_B: now also R51.1
- net at U1.34 (RXD0/IO3): now also R49.1; no longer J3.2 (Pin_2)
- net at U1.35 (TXD0/IO1): now also R48.1; no longer J3.1 (Pin_1)
- new net: D4.2 (A), R52.2
- new net: J3.1 (Pin_1), R48.2
- new net: J3.2 (Pin_2), R49.2
- new net: D3.2 (A), R51.2
- no-connect marks 19 -> 17
Other:
- moved on the sheet: C23
