File: feedback.kicad_sch (KiCad schematic)
At the start: 15 parts, among them U4 TLV9001IDCK

Commit message: Start layout
Parts:
- C35, C36: value 10n -> 1n; LCSC C57112 -> C1588
- R2, R3, R4, R5: value 1k -> 10k; LCSC C21190 -> C25804
Changed lines of the file:
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@@
 			)
 		)
-		(property "Value" "1k"
+		(property "Value" "10k"
 			(at 147.32 106.68 90)
 			(effects
@@
 			)
 		)
-		(property "LCSC" "C21190"
+		(property "LCSC" "C25804"
 			(at 147.32 109.22 0)
 			(effects
@@
 			)
 		)
-		(property "Value" "10n"
+		(property "Value" "1n"
 			(at 127 85.0835 0)
 			(effects
@@
 			)
 		)
-		(property "LCSC" "C57112"
+		(property "LCSC" "C1588"
 			(at 124.46 83.82 0)
 			(effects
@@
 			)
 		)
-		(property "Value" "10n"
+		(property "Value" "1n"
 			(at 147.3263 118.11 90)
 			(effects
@@
 			)
 		)
-		(property "LCSC" "C57112"
+		(property "LCSC" "C1588"
 			(at 147.32 121.92 0)
 			(effects
@@
 			)
 		)
-		(property "Value" "1k"
+		(property "Value" "10k"
 			(at 106.68 91.44 90)
 			(effects
@@
 			)
 		)
-		(property "LCSC" "C21190"
+		(property "LCSC" "C25804"
 			(at 106.68 91.44 0)
 			(effects
@@
 			)
 		)
-		(property "Value" "1k"
+		(property "Value" "10k"
 			(at 106.68 96.52 90)
 			(effects
@@
 			)
 		)
-		(property "LCSC" "C21190"
+		(property "LCSC" "C25804"
 			(at 106.68 96.52 0)
 			(effects
@@
 			)
 		)
-		(property "Value" "1k"
+		(property "Value" "10k"
 			(at 135.89 85.0899 0)
 			(effects
@@
 			)
 		)
-		(property "LCSC" "C21190"
+		(property "LCSC" "C25804"
 			(at 138.43 83.82 0)
 			(effects

Commit message: Manufacturing update + inductor fix
Parts:
- U4: JLCPCB_CORRECTION (none) -> 0;0;270; LCSC (none) -> C398362
Changed lines of the file:
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@@
+			)
+		)
+		(property "LCSC" "C398362"
+			(at 146.05 93.98 0)
+			(effects
+				(font
+					(size 1.27 1.27)
+				)
+				(hide yes)
+			)
+		)
+		(property "JLCPCB_CORRECTION" "0;0;270"
+			(at 146.05 93.98 0)
+			(effects
+				(font
+					(size 1.27 1.27)
+				)
+				(hide yes)
 			)
 		)
