File: internal_power.kicad_sch (KiCad schematic)
At the start: 15 parts, among them U6 LMR51450F

Commit message: Routing almost finished
Parts:
- added C13: 10u, Capacitor_SMD:C_1206_3216Metric, symbol Device:C
- added C14: 47u, Capacitor_SMD:C_1206_3216Metric, symbol Device:C
- added L4: 4.7uH (SWPA5020S4R7MT), Inductor_SMD:L_Sunlord_SWPA5020S, symbol Device:L
- added R50: 1, Resistor_SMD:R_0603_1608Metric, symbol rflib:R
Connections:
- net GND: now also C13.2, C14.2
- net V_{out}: now also C13.1, L4.2, R50.1; no longer C29.1, C30.1, L2.2
- net SW: now reaches C28.2, L2.1, U6.1 (SW), U6.2 (SW), U6.3 (SW)
- net SW: no longer C31.1, R29.1
- new net: C14.1, R50.2
- new net 3V3_UNFILT: C29.1, C30.1, C31.1, L2.2, L4.1, R29.1
Other:
- moved on the sheet: C31, D2, L2, R29, R30, R32, TP10

Commit message: Manufacturing update + inductor fix
Parts:
- TP10: LCSC C5199804 -> (none)
Changed lines of the file:
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@@
-			)
-		)
-		(property "LCSC" "C5199804"
-			(at 245.11 87.63 0)
-			(effects
-				(font
-					(size 1.27 1.27)
-				)
-				(hide yes)
 			)
 		)
