File: pwm_reject.kicad_sch (KiCad schematic)
At the start: 16 parts, among them U3 TLV9001IDCK, U5 TLV9001IDCK

Commit message: Start layout
Parts:
- added R46: 100k, Resistor_SMD:R_0603_1608Metric, symbol rflib:R
Connections:
- net GND: now also R1.2, R46.1; no longer R6.1
- net at R39.2, R44.2, U3.1 (+): now also R46.2
- net at C3.1, R10.1, R9.2: now also R6.2; no longer R1.1
- new net: R1.1, R6.1
Other:
- note added: "This may be needed to nullify offset somewhere"
- moved on the sheet: R1, R6
Changed lines of the file:
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@@
+	(wire
+		(pts
+			(xy 185.42 95.25) (xy 185.42 102.87)
+		)
+		(stroke
+			(width 0)
+			(type default)
+		)
+	)
 	(wire
 		(pts
@@
 	(wire
 		(pts
-			(xy 124.46 85.09) (xy 128.27 85.09)
+			(xy 185.42 110.49) (xy 185.42 111.76)
 		)
 		(stroke
@@
 	(wire
 		(pts
-			(xy 160.02 93.98) (xy 160.02 95.25)
+			(xy 124.46 85.09) (xy 128.27 85.09)
 		)
 		(stroke
@@
 	(wire
 		(pts
-			(xy 207.01 100.33) (xy 213.36 100.33)
+			(xy 160.02 93.98) (xy 160.02 95.25)
 		)
 		(stroke
 			(width 0)
 			(type default)
+		)
+	)
+	(wire
+		(pts
+			(xy 207.01 100.33) (xy 213.36 100.33)
+		)
+		(stroke
+			(width 0)
+			(type default)
+		)
+	)
+	(text "This may be needed to nullify offset somewhere"
+		(exclude_from_sim no)
+		(at 172.212 116.84 0)
+		(effects
+			(font
+				(size 1.27 1.27)
+			)
 		)
 	)
@@
 	(text "Pot sets maximum current"
 		(exclude_from_sim no)
-		(at 70.866 100.076 0)
+		(at 58.42 99.06 0)
 		(effects
 			(font
@@
 	)
 	(symbol
+		(lib_id "rflib:R")
+		(at 185.42 106.68 180)
+		(unit 1)
+		(exclude_from_sim no)
+		(in_bom yes)
+		(on_board yes)
+		(dnp yes)
+		(property "Reference" "R46"
+			(at 182.88 107.95 0)
+			(effects
+				(font
+					(size 1.27 1.27)
+				)
+				(justify left)
+			)
+		)
+		(property "Value" "100k"
+			(at 181.61 105.41 0)
+			(effects
+				(font
+					(size 1.27 1.27)
+				)
+			)
+		)
+		(property "Footprint" "Resistor_SMD:R_0603_1608Metric"
+			(at 187.198 106.68 90)
+			(effects
+				(font
+					(size 1.27 1.27)
+				)
+				(hide yes)
+			)
+		)
+		(property "Datasheet" "~"
+			(at 185.42 106.68 0)
+			(effects
+				(font
+					(size 1.27 1.27)
+				)
+				(hide yes)
+			)
+		)
+		(property "Description" "Resistor"
+			(at 185.42 106.68 0)
+			(effects
+				(font
+					(size 1.27 1.27)
+				)
+				(hide yes)
+			)
+		)
+		(property "Manufacturer_Name" ""
+			(at 185.42 106.68 0)
+			(effects
+				(font
+					(size 1.27 1.27)
+				)
+				(hide yes)
+			)
+		)
+		(property "Manufacturer_Part_Number" ""
+			(at 185.42 106.68 0)
+			(effects
+				(font
+					(size 1.27 1.27)
+				)
+				(hide yes)
+			)
+		)
+		(property "JLCPCB_CORRECTION" ""
+			(at 185.42 106.68 0)
+			(effects
+				(font
+					(size 1.27 1.27)
+				)
+				(hide yes)
+			)
+		)
+		(property "Arrow Part Number" ""
+			(at 185.42 106.68 0)
+			(effects
+				(font
+					(size 1.27 1.27)
+				)
+				(hide yes)
+			)
+		)
+		(property "Arrow Price/Stock" ""
+			(at 185.42 106.68 0)
+			(effects
+				(font
+					(size 1.27 1.27)
+				)
+				(hide yes)
+			)
+		)
+		(pin "1"
+		)
+		(pin "2"
+		)
+		(instances
+			(project "silence"
+				(path "/fe89ff8c-41b6-4857-bb57-156cc6b22e44/3f3de578-1b7e-481d-ab2d-91c68c64d542/3f3d567a-1187-4bed-9774-f365abfa2a84"
+					(reference "R46")
+					(unit 1)
+				)
+			)
+		)
+	)
+	(symbol
 		(lib_id "power:GND")
 		(at 124.46 102.87 0)
@@
 	)
 	(symbol
+		(lib_id "power:GND")
+		(at 185.42 111.76 0)
+		(unit 1)
+		(exclude_from_sim no)
+		(in_bom yes)
+		(on_board yes)
+		(dnp no)
+		(fields_autoplaced yes)
+		(property "Reference" "#PWR093"
+			(at 185.42 118.11 0)
+			(effects
+				(font
+					(size 1.27 1.27)
+				)
+				(hide yes)
+			)
+		)
+		(property "Value" "GND"
+			(at 185.42 116.84 0)
+			(effects
+				(font
+					(size 1.27 1.27)
+				)
+				(hide yes)
+			)
+		)
+		(property "Footprint" ""
+			(at 185.42 111.76 0)
+			(effects
+				(font
+					(size 1.27 1.27)
+				)
+				(hide yes)
+			)
+		)
+		(property "Datasheet" ""
+			(at 185.42 111.76 0)
+			(effects
+				(font
+					(size 1.27 1.27)
+				)
+				(hide yes)
+			)
+		)
+		(property "Description" "Power symbol creates a global label with name \"GND\" , ground"
+			(at 185.42 111.76 0)
+			(effects
+				(font
+					(size 1.27 1.27)
+				)
+				(hide yes)
+			)
+		)
+		(pin "1"
+		)
+		(instances
+			(project "silence"
+				(path "/fe89ff8c-41b6-4857-bb57-156cc6b22e44/3f3de578-1b7e-481d-ab2d-91c68c64d542/3f3d567a-1187-4bed-9774-f365abfa2a84"
+					(reference "#PWR093")
+					(unit 1)
+				)
+			)
+		)
+	)
+	(symbol
 		(lib_id "rflib:R")
 		(at 106.68 92.71 90)
@@
 	(symbol
 		(lib_id "rflib:R")
-		(at 87.63 107.95 180)
+		(at 87.63 99.06 180)
 		(unit 1)
 		(exclude_from_sim no)
@@
 		(dnp no)
 		(property "Reference" "R6"
-			(at 85.09 109.22 0)
+			(at 85.09 100.33 0)
 			(effects
 				(font
@@
 		)
 		(property "Value" "100"
-			(at 83.82 106.68 0)
+			(at 83.82 97.79 0)
 			(effects
 				(font
@@
 		)
 		(property "Footprint" "Resistor_SMD:R_0603_1608Metric"
-			(at 89.408 107.95 90)
+			(at 89.408 99.06 90)
 			(effects
 				(font
@@
 		)
 		(property "Datasheet" "~"
-			(at 87.63 107.95 0)
+			(at 87.63 99.06 0)
 			(effects
 				(font
@@
 		)
 		(property "Description" "Resistor"
-			(at 87.63 107.95 0)
+			(at 87.63 99.06 0)
 			(effects
 				(font
@@
 		)
 		(property "LCSC" "C25804"
-			(at 87.63 107.95 0)
+			(at 87.63 99.06 0)
 			(effects
 				(font
@@
 		)
 		(property "Manufacturer_Name" ""
-			(at 87.63 107.95 0)
+			(at 87.63 99.06 0)
 			(effects
 				(font
@@
 		)
 		(property "Manufacturer_Part_Number" ""
-			(at 87.63 107.95 0)
+			(at 87.63 99.06 0)
 			(effects
 				(font
@@
 		)
 		(property "JLCPCB_CORRECTION" ""
-			(at 87.63 107.95 0)
+			(at 87.63 99.06 0)
 			(effects
 				(font
@@
 		)
 		(property "Arrow Part Number" ""
-			(at 87.63 107.95 0)
+			(at 87.63 99.06 0)
 			(effects
 				(font
@@
 		)
 		(property "Arrow Price/Stock" ""
-			(at 87.63 107.95 0)
+			(at 87.63 99.06 0)
 			(effects
 				(font
@@
 	(symbol
 		(lib_id "Device:R_Variable")
-		(at 87.63 99.06 0)
+		(at 87.63 107.95 0)
 		(unit 1)
 		(exclude_from_sim no)
@@
 		(fields_autoplaced yes)
 		(property "Reference" "R1"
-			(at 91.44 97.7899 0)
+			(at 91.44 106.6799 0)
 			(effects
 				(font
@@
 		)
 		(property "Value" "10k"
-			(at 91.44 100.3299 0)
+			(at 91.44 109.2199 0)
 			(effects
 				(font
@@
 		)
 		(property "Footprint" "Potentiometer_THT:Potentiometer_Bourns_3296W_Vertical"
-			(at 85.852 99.06 90)
+			(at 85.852 107.95 90)
 			(effects
 				(font
@@
 		)
 		(property "Datasheet" "~"
-			(at 87.63 99.06 0)
+			(at 87.63 107.95 0)
 			(effects
 				(font
@@
 		)
 		(property "Description" "Variable resistor"
-			(at 87.63 99.06 0)
-			(effects
-				(font
+			(at 87.63 107.95 0)
+			(effects
+				(font

Commit message: Manufacturing update + inductor fix
Parts:
- U3, U5: JLCPCB_CORRECTION (none) -> 0;0;270; LCSC (none) -> C398362
Changed lines of the file:
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@@
+			)
+		)
+		(property "LCSC" "C398362"
+			(at 124.46 95.25 0)
+			(effects
+				(font
+					(size 1.27 1.27)
+				)
+				(hide yes)
+			)
+		)
+		(property "JLCPCB_CORRECTION" "0;0;270"
+			(at 124.46 95.25 0)
+			(effects
+				(font
+					(size 1.27 1.27)
+				)
+				(hide yes)
 			)
 		)
@@
 			(at 218.44 97.79 0)
 			(effects
+				(font
+					(size 1.27 1.27)
+				)
+				(hide yes)
+			)
+		)
+		(property "LCSC" "C398362"
+			(at 218.44 97.79 0)
+			(effects
+				(font
+					(size 1.27 1.27)
+				)
+				(hide yes)
+			)
+		)
+		(property "JLCPCB_CORRECTION" "0;0;270"
+			(at 218.44 97.79 0)
+			(effects
