File: silence.kicad_sch (KiCad schematic)
At the start: 7 parts, among them J1 15EDGVC-3.81-02P, J2 15EDGVC-2.5-04P-14, J5 15EDGVC-3.81-02P

Commit message: Routing almost finished
Parts:
- added D5: LED, LED_SMD:LED_0603_1608Metric, symbol Device:LED
- added R53: 47k, Resistor_SMD:R_0603_1608Metric, symbol rflib:R
Connections:
- net +VDC: now also R53.1
- net GND: now also D5.1 (K)
- new net: D5.2 (A), R53.2

Commit message: Minor edits
Parts:
- added TP12: VDC, meteopress_footprints:TestPoint_THTPad_D2.0mm_Drill1.0mm, symbol Connector:TestPoint
Connections:
- net +VDC: now also TP12.1
Changed lines of the file:
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@@
+	)
+	(junction
+		(at 72.39 64.77)
+		(diameter 0)
+		(color 0 0 0 0)
 	)
 	(junction
@@
 	(wire
 		(pts
+			(xy 72.39 64.77) (xy 81.28 64.77)
+		)
+		(stroke
+			(width 0)
+			(type default)
+		)
+	)
+	(wire
+		(pts
+			(xy 72.39 62.23) (xy 72.39 64.77)
+		)
+		(stroke
+			(width 0)
+			(type default)
+		)
+	)
+	(wire
+		(pts
 			(xy 128.27 76.2) (xy 128.27 91.44)
 		)
@@
 	(wire
 		(pts
-			(xy 67.31 64.77) (xy 81.28 64.77)
+			(xy 67.31 64.77) (xy 72.39 64.77)
 		)
 		(stroke
@@
 					(unit 1)
 				)
+			)
+		)
+	)
+	(symbol
+		(lib_id "Connector:TestPoint")
+		(at 72.39 62.23 0)
+		(unit 1)
+		(exclude_from_sim no)
+		(in_bom yes)
+		(on_board yes)
+		(dnp no)
+		(fields_autoplaced yes)
+		(property "Reference" "TP12"
+			(at 74.93 57.6579 0)
+			(effects
+				(font
+					(size 1.27 1.27)
+				)
+				(justify left)
+			)
+		)
+		(property "Value" "VDC"
+			(at 74.93 60.1979 0)
+			(effects
+				(font
+					(size 1.27 1.27)
+				)
+				(justify left)
+			)
+		)
+		(property "Footprint" "meteopress_footprints:TestPoint_THTPad_D2.0mm_Drill1.0mm"
+			(at 77.47 62.23 0)
+			(effects
+				(font
+					(size 1.27 1.27)
+				)
+				(hide yes)
+			)
+		)
+		(property "Datasheet" "~"
+			(at 77.47 62.23 0)
+			(effects
+				(font
+					(size 1.27 1.27)
+				)
+				(hide yes)
+			)
+		)
+		(property "Description" "test point"
+			(at 72.39 62.23 0)
+			(effects
+				(font
+					(size 1.27 1.27)
+				)
+				(hide yes)
+			)
+		)
+		(property "LCSC" "C5199804"
+			(at 72.39 62.23 0)
+			(effects
+				(font
+					(size 1.27 1.27)
+				)
+				(hide yes)
+			)
+		)
+		(pin "1"
+		)
+		(instances
+			(project "silence"
+				(path "/fe89ff8c-41b6-4857-bb57-156cc6b22e44"
+					(reference "TP12")
+					(unit 1)
+				)

Commit message: Manufacturing update + inductor fix
Parts:
- TP12: LCSC C5199804 -> (none)
Changed lines of the file:
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@@
-			)
-		)
-		(property "LCSC" "C5199804"
-			(at 72.39 62.23 0)
-			(effects
-				(font
-					(size 1.27 1.27)
-				)
-				(hide yes)
 			)
 		)
