File: voff_source.kicad_sch (KiCad schematic)
At the start: 10 parts, among them U8 TLV9001IDCK

Commit message: Minor updates
Parts:
- added R47: 0, Resistor_SMD:R_0603_1608Metric, symbol rflib:R
Connections:
- net GND: now also R41.2; no longer R42.2
- net at R42.1: now also C41.1, R40.1, U8.1 (+); no longer R41.2
- net at FB2.1, U8.4: now also R47.2; no longer U8.3 (-)
- new net: R47.1, U8.3 (-)
- new net: R41.1, R42.2
Other:
- moved on the sheet: R41, R42
Changed lines of the file:
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@@
+	(wire
+		(pts
+			(xy 144.78 119.38) (xy 152.4 119.38)
+		)
+		(stroke
+			(width 0)
+			(type default)
+		)
+	)
 	(wire
 		(pts
@@
 	(wire
 		(pts
-			(xy 128.27 119.38) (xy 152.4 119.38)
+			(xy 128.27 119.38) (xy 137.16 119.38)
 		)
 		(stroke
@@
 	)
 	(symbol
+		(lib_id "rflib:R")
+		(at 140.97 119.38 90)
+		(unit 1)
+		(exclude_from_sim no)
+		(in_bom yes)
+		(on_board yes)
+		(dnp no)
+		(fields_autoplaced yes)
+		(property "Reference" "R47"
+			(at 140.97 123.19 90)
+			(effects
+				(font
+					(size 1.27 1.27)
+				)
+			)
+		)
+		(property "Value" "0"
+			(at 140.97 125.73 90)
+			(effects
+				(font
+					(size 1.27 1.27)
+				)
+			)
+		)
+		(property "Footprint" "Resistor_SMD:R_0603_1608Metric"
+			(at 140.97 121.158 90)
+			(effects
+				(font
+					(size 1.27 1.27)
+				)
+				(hide yes)
+			)
+		)
+		(property "Datasheet" "~"
+			(at 140.97 119.38 0)
+			(effects
+				(font
+					(size 1.27 1.27)
+				)
+				(hide yes)
+			)
+		)
+		(property "Description" "Resistor"
+			(at 140.97 119.38 0)
+			(effects
+				(font
+					(size 1.27 1.27)
+				)
+				(hide yes)
+			)
+		)
+		(property "LCSC" "C15402"
+			(at 140.97 119.38 0)
+			(effects
+				(font
+					(size 1.27 1.27)
+				)
+				(hide yes)
+			)
+		)
+		(property "Manufacturer_Name" ""
+			(at 140.97 119.38 0)
+			(effects
+				(font
+					(size 1.27 1.27)
+				)
+				(hide yes)
+			)
+		)
+		(property "Manufacturer_Part_Number" ""
+			(at 140.97 119.38 0)
+			(effects
+				(font
+					(size 1.27 1.27)
+				)
+				(hide yes)
+			)
+		)
+		(property "Arrow Part Number" ""
+			(at 140.97 119.38 0)
+			(effects
+				(font
+					(size 1.27 1.27)
+				)
+				(hide yes)
+			)
+		)
+		(property "Arrow Price/Stock" ""
+			(at 140.97 119.38 0)
+			(effects
+				(font
+					(size 1.27 1.27)
+				)
+				(hide yes)
+			)
+		)
+		(pin "1"
+		)
+		(pin "2"
+		)
+		(instances
+			(project "silence"
+				(path "/fe89ff8c-41b6-4857-bb57-156cc6b22e44/5a17d479-20e3-4170-9c0f-6c7b7ade91f6"
+					(reference "R47")
+					(unit 1)
+				)
+			)
+		)
+	)
+	(symbol
 		(lib_id "power:+3V3")
 		(at 30.48 27.94 0)
@@
 	(symbol
 		(lib_id "rflib:R")
-		(at 109.22 114.3 0)
+		(at 109.22 106.68 0)
 		(unit 1)
 		(exclude_from_sim no)
@@
 		(fields_autoplaced yes)
 		(property "Reference" "R42"
-			(at 111.76 113.0299 0)
+			(at 111.76 105.4099 0)
 			(effects
 				(font
@@
 		)
 		(property "Value" "1k"
-			(at 111.76 115.5699 0)
+			(at 111.76 107.9499 0)
 			(effects
 				(font
@@
 		)
 		(property "Footprint" "Resistor_SMD:R_0603_1608Metric"
-			(at 107.442 114.3 90)
+			(at 107.442 106.68 90)
 			(effects
 				(font
@@
 		)
 		(property "Datasheet" "~"
-			(at 109.22 114.3 0)
+			(at 109.22 106.68 0)
 			(effects
 				(font
@@
 		)
 		(property "Description" "Resistor"
-			(at 109.22 114.3 0)
+			(at 109.22 106.68 0)
 			(effects
 				(font
@@
 		)
 		(property "LCSC" "C21190"
-			(at 109.22 114.3 0)
+			(at 109.22 106.68 0)
 			(effects
 				(font
@@
 		)
 		(property "Manufacturer_Name" ""
-			(at 109.22 114.3 0)
+			(at 109.22 106.68 0)
 			(effects
 				(font
@@
 		)
 		(property "Manufacturer_Part_Number" ""
-			(at 109.22 114.3 0)
+			(at 109.22 106.68 0)
 			(effects
 				(font
@@
 		)
 		(property "Arrow Part Number" ""
-			(at 109.22 114.3 0)
+			(at 109.22 106.68 0)
 			(effects
 				(font
@@
 		)
 		(property "Arrow Price/Stock" ""
-			(at 109.22 114.3 0)
+			(at 109.22 106.68 0)
 			(effects
 				(font
@@
 	(symbol
 		(lib_id "Device:R_Variable")
-		(at 109.22 106.68 0)
+		(at 109.22 114.3 0)
 		(unit 1)
 		(exclude_from_sim no)
@@
 		(fields_autoplaced yes)
 		(property "Reference" "R41"
-			(at 113.03 105.4099 0)
+			(at 113.03 113.0299 0)
 			(effects
 				(font
@@
 		)
 		(property "Value" "10k"
-			(at 113.03 107.9499 0)
+			(at 113.03 115.5699 0)
 			(effects
 				(font
@@
 		)
 		(property "Footprint" "Potentiometer_THT:Potentiometer_Bourns_3296W_Vertical"
-			(at 107.442 106.68 90)
+			(at 107.442 114.3 90)
 			(effects
 				(font
@@
 		)
 		(property "Datasheet" "~"
-			(at 109.22 106.68 0)
+			(at 109.22 114.3 0)
 			(effects
 				(font
@@
 		)
 		(property "Description" "Variable resistor"
-			(at 109.22 106.68 0)
-			(effects
-				(font
+			(at 109.22 114.3 0)
+			(effects
+				(font

Commit message: Manufacturing update + inductor fix
Parts:
- FB2: LCSC (none) -> C1002
- R47: LCSC C15402 -> C21189
- TP13: LCSC C5199804 -> (none)
- U8: JLCPCB_CORRECTION (none) -> 0;0;270; LCSC (none) -> C398362
Changed lines of the file:
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@@
-			)
-		)
-		(property "LCSC" "C5199804"
-			(at 189.23 102.87 0)
-			(effects
-				(font
-					(size 1.27 1.27)
-				)
-				(hide yes)
 			)
 		)
@@
 			)
 		)
-		(property "LCSC" "C15402"
+		(property "LCSC" "C21189"
 			(at 140.97 119.38 0)
 			(effects
@@
 			)
 		)
+		(property "LCSC" "C398362"
+			(at 139.7 104.14 0)
+			(effects
+				(font
+					(size 1.27 1.27)
+				)
+				(hide yes)
+			)
+		)
+		(property "JLCPCB_CORRECTION" "0;0;270"
+			(at 139.7 104.14 0)
+			(effects
+				(font
+					(size 1.27 1.27)
+				)
+				(hide yes)
+			)
+		)
 		(pin "4"
 		)
@@
 			(effects
 				(font
+					(size 1.27 1.27)
+				)
+				(hide yes)
+			)
+		)
+		(property "LCSC" "C1002"
+			(at 170.18 104.14 90)
+			(effects
+				(font
