File: vref_filter.kicad_sch (KiCad schematic)
At the start: 6 parts

Commit message: Manufacturing update + inductor fix
Parts:
- TP9: LCSC C5199804 -> (none)
Changed lines of the file:
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@@
-			)
-		)
-		(property "LCSC" "C5199804"
-			(at 157.48 86.36 0)
-			(effects
-				(font
-					(size 1.27 1.27)
-				)
-				(hide yes)
 			)
 		)
