File: ws2812.kicad_sch (KiCad schematic)
At the start: 11 parts, among them Q2 AO3400A

Commit message: Start layout
Parts:
- gave numbers to parts that had none: 3
Changed lines of the file:
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@@
 		(dnp no)
 		(fields_autoplaced yes)
-		(property "Reference" "#PWR?"
+		(property "Reference" "#PWR0101"
 			(at 105.41 87.63 0)
 			(effects
@@
 			(project "silence"
 				(path "/fe89ff8c-41b6-4857-bb57-156cc6b22e44/247c4e69-048b-4eca-aae5-8cfe880c7ffc"
-					(reference "#PWR?")
+					(reference "#PWR0101")
 					(unit 1)
 				)
@@
 		(dnp no)
 		(fields_autoplaced yes)
-		(property "Reference" "Q?"
+		(property "Reference" "Q1"
 			(at 109.22 101.5999 0)
 			(effects
@@
 			(project "silence"
 				(path "/fe89ff8c-41b6-4857-bb57-156cc6b22e44/247c4e69-048b-4eca-aae5-8cfe880c7ffc"
-					(reference "Q?")
+					(reference "Q1")
 					(unit 1)
 				)
@@
 		(dnp no)
 		(fields_autoplaced yes)
-		(property "Reference" "TP?"
+		(property "Reference" "TP15"
 			(at 88.9 94.4879 0)
 			(effects
@@
 			(project "silence"
 				(path "/fe89ff8c-41b6-4857-bb57-156cc6b22e44/247c4e69-048b-4eca-aae5-8cfe880c7ffc"
-					(reference "TP?")
+					(reference "TP15")
 					(unit 1)
 				)
@@
 		(dnp no)
 		(fields_autoplaced yes)
-		(property "Reference" "J?"
+		(property "Reference" "J7"
 			(at 227.33 95.2499 0)
 			(effects
@@
 			(project "silence"
 				(path "/fe89ff8c-41b6-4857-bb57-156cc6b22e44/247c4e69-048b-4eca-aae5-8cfe880c7ffc"
-					(reference "J?")
-					(unit 1)
-				)
+					(reference "J7")
+					(unit 1)
+				)

Commit message: Routing almost finished
Parts:
- added JP4: WSEN, Jumper:SolderJumper-2_P1.3mm_Open_RoundedPad1.0x1.5mm, symbol Jumper:SolderJumper_2_Open
- TP3: value DIN -> DO
Connections:
- net +VDC: now also JP4.2 (B); no longer R12.1, R15.1
- new net: JP4.1 (A), R12.1, R15.1
Other:
- note added: "Beware that these FETs are only rated up to 30V So this part is disabled by default and should be enabled only on boards that are powered from +5V"
Changed lines of the file:
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@@
+	)
+	(junction
+		(at 105.41 82.55)
+		(diameter 0)
+		(color 0 0 0 0)
 	)
 	(junction
@@
 	(wire
 		(pts
+			(xy 105.41 72.39) (xy 105.41 71.12)
+		)
+		(stroke
+			(width 0)
+			(type default)
+		)
+	)
+	(wire
+		(pts
 			(xy 92.71 102.87) (xy 92.71 105.41)
 		)
@@
 	(wire
 		(pts
-			(xy 165.1 85.09) (xy 165.1 87.63)
-		)
-		(stroke
-			(width 0)
-			(type default)
-		)
-	)
-	(wire
-		(pts
 			(xy 152.4 114.3) (xy 152.4 113.03)
 		)
@@
 	(wire
 		(pts
+			(xy 165.1 82.55) (xy 165.1 87.63)
+		)
+		(stroke
+			(width 0)
+			(type default)
+		)
+	)
+	(wire
+		(pts
 			(xy 205.74 96.52) (xy 205.74 100.33)
 		)
@@
 	(wire
 		(pts
-			(xy 105.41 85.09) (xy 105.41 87.63)
+			(xy 105.41 82.55) (xy 105.41 87.63)
 		)
 		(stroke
@@
 	(wire
 		(pts
+			(xy 105.41 82.55) (xy 165.1 82.55)
+		)
+		(stroke
+			(width 0)
+			(type default)
+		)
+	)
+	(wire
+		(pts
 			(xy 152.4 102.87) (xy 152.4 105.41)
 		)
@@
 		(pts
 			(xy 205.74 96.52) (xy 220.98 96.52)
+		)
+		(stroke
+			(width 0)
+			(type default)
+		)
+	)
+	(wire
+		(pts
+			(xy 105.41 80.01) (xy 105.41 82.55)
 		)
 		(stroke
@@
 				(size 1.27 1.27)
 			)
+		)
+	)
+	(text "Beware that these FETs are only rated up to 30V\nSo this part is disabled by default and should be enabled only on boards that are powered from +5V"
+		(exclude_from_sim no)
+		(at 114.808 76.2 0)
+		(effects
+			(font
+				(size 1.27 1.27)
+			)
+			(justify left)
 		)
 	)
@@
 	)
 	(symbol
-		(lib_id "power:+VDC")
-		(at 165.1 85.09 0)
-		(unit 1)
-		(exclude_from_sim no)
-		(in_bom yes)
-		(on_board yes)
-		(dnp no)
-		(fields_autoplaced yes)
-		(property "Reference" "#PWR025"
-			(at 165.1 87.63 0)
-			(effects
-				(font
-					(size 1.27 1.27)
-				)
-				(hide yes)
-			)
-		)
-		(property "Value" "+VDC"
-			(at 165.1 77.47 0)
-			(effects
-				(font
-					(size 1.27 1.27)
-				)
-			)
-		)
-		(property "Footprint" ""
-			(at 165.1 85.09 0)
-			(effects
-				(font
-					(size 1.27 1.27)
-				)
-				(hide yes)
-			)
-		)
-		(property "Datasheet" ""
-			(at 165.1 85.09 0)
-			(effects
-				(font
-					(size 1.27 1.27)
-				)
-				(hide yes)
-			)
-		)
-		(property "Description" "Power symbol creates a global label with name \"+VDC\""
-			(at 165.1 85.09 0)
-			(effects
-				(font
-					(size 1.27 1.27)
-				)
-				(hide yes)
-			)
-		)
-		(pin "1"
-		)
-		(instances
-			(project "silence"
-				(path "/fe89ff8c-41b6-4857-bb57-156cc6b22e44/247c4e69-048b-4eca-aae5-8cfe880c7ffc"
-					(reference "#PWR025")
-					(unit 1)
-				)
-				(path "/fe89ff8c-41b6-4857-bb57-156cc6b22e44/fede6b6b-db35-4020-9cfa-2ae12bdfcee5"
-					(reference "#PWR029")
-					(unit 1)
-				)
-			)
-		)
-	)
-	(symbol
 		(lib_id "rflib:R")
 		(at 198.12 96.52 90)
@@
 	(symbol
 		(lib_id "power:+VDC")
-		(at 105.41 85.09 0)
+		(at 105.41 71.12 0)
 		(unit 1)
 		(exclude_from_sim no)
@@
 		(fields_autoplaced yes)
 		(property "Reference" "#PWR0101"
-			(at 105.41 87.63 0)
+			(at 105.41 73.66 0)
 			(effects
 				(font
@@
 		)
 		(property "Value" "+VDC"
-			(at 105.41 77.47 0)
+			(at 105.41 63.5 0)
 			(effects
 				(font
@@
 		)
 		(property "Footprint" ""
-			(at 105.41 85.09 0)
+			(at 105.41 71.12 0)
 			(effects
 				(font
@@
 		)
 		(property "Datasheet" ""
-			(at 105.41 85.09 0)
+			(at 105.41 71.12 0)
 			(effects
 				(font
@@
 		)
 		(property "Description" "Power symbol creates a global label with name \"+VDC\""
-			(at 105.41 85.09 0)
+			(at 105.41 71.12 0)
 			(effects
 				(font
@@
 	)
 	(symbol
+		(lib_id "Jumper:SolderJumper_2_Open")
+		(at 105.41 76.2 90)
+		(unit 1)
+		(exclude_from_sim yes)
+		(in_bom no)
+		(on_board yes)
+		(dnp no)
+		(fields_autoplaced yes)
+		(property "Reference" "JP4"
+			(at 107.95 74.9299 90)
+			(effects
+				(font
+					(size 1.27 1.27)
+				)
+				(justify right)
+			)
+		)
+		(property "Value" "WSEN"
+			(at 107.95 77.4699 90)
+			(effects
+				(font
+					(size 1.27 1.27)
+				)
+				(justify right)
+			)
+		)
+		(property "Footprint" "Jumper:SolderJumper-2_P1.3mm_Open_RoundedPad1.0x1.5mm"
+			(at 105.41 76.2 0)
+			(effects
+				(font
+					(size 1.27 1.27)
+				)
+				(hide yes)
+			)
+		)
+		(property "Datasheet" "~"
+			(at 105.41 76.2 0)
+			(effects
+				(font
+					(size 1.27 1.27)
+				)
+				(hide yes)
+			)
+		)
+		(property "Description" "Solder Jumper, 2-pole, open"
+			(at 105.41 76.2 0)
+			(effects
+				(font
+					(size 1.27 1.27)
+				)
+				(hide yes)
+			)
+		)
+		(pin "2"
+		)
+		(pin "1"
+		)
+		(instances
+			(project ""
+				(path "/fe89ff8c-41b6-4857-bb57-156cc6b22e44/247c4e69-048b-4eca-aae5-8cfe880c7ffc"
+					(reference "JP4")
+					(unit 1)
+				)
+				(path "/fe89ff8c-41b6-4857-bb57-156cc6b22e44/fede6b6b-db35-4020-9cfa-2ae12bdfcee5"
+					(reference "JP3")
+					(unit 1)
+				)
+			)
+		)
+	)
+	(symbol
 		(lib_id "rflib:R")
 		(at 184.15 106.68 0)
@@
 			)
 		)
-		(property "Value" "DIN"
+		(property "Value" "DO"
 			(at 208.28 104.9019 0)
 			(effects

Commit message: Minor updates
Parts:
- removed JP4: WSEN, Jumper:SolderJumper-2_P1.3mm_Open_RoundedPad1.0x1.5mm, symbol Jumper:SolderJumper_2_Open
- removed Q1, Q2: AO3400A, Package_TO_SOT_SMD:SOT-23, symbol Transistor_FET:AO3400A
- removed R13, R14: 1M, Resistor_SMD:R_0603_1608Metric, symbol rflib:R
- added Q1, Q6: MMBT5551L, Package_TO_SOT_SMD:SOT-23, symbol Transistor_BJT:MMBT5551L
- added R54: 10k, Resistor_SMD:R_0603_1608Metric, symbol rflib:R
Connections:
- net +VDC: now also R12.1, R15.1
- net DIN: now also R54.1
- net GND: now also Q1.2 (E), Q6.2 (E)
- net at R15.2, R16.1, R37.1: now also Q1.3 (C)
- net at R12.2: now also Q1.1 (B), Q6.3 (C)
- new net: Q6.1 (B), R54.2
Other:
- note removed: "Beware that these FETs are only rated up to 30V So this part is disabled by default and should be enabled only on boards that are powered from +5V"
- note removed: "TODO: Connector type"
- moved on the sheet: TP15

Commit message: Minor edits
Parts:
- renumbered Q1 to Q3, R54 to R55
Changed lines of the file:
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@@
 		(dnp no)
 		(fields_autoplaced yes)
-		(property "Reference" "Q1"
+		(property "Reference" "Q3"
 			(at 167.64 101.5999 0)
 			(effects
@@
 		(dnp no)
 		(fields_autoplaced yes)
-		(property "Reference" "R54"
+		(property "Reference" "R55"
 			(at 81.28 96.52 90)
 			(effects

Commit message: Manufacturing update + inductor fix
Parts:
- Q3, Q6: JLCPCB_CORRECTION (none) -> 0;0;180
Changed lines of the file:
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@@
+			)
+		)
+		(property "JLCPCB_CORRECTION" "0;0;180"
+			(at 162.56 102.87 0)
+			(effects
+				(font
+					(size 1.27 1.27)
+				)
+				(hide yes)
 			)
 		)
@@
 			(at 102.87 102.87 0)
 			(effects
+				(font
+					(size 1.27 1.27)
+				)
+				(hide yes)
+			)
+		)
+		(property "JLCPCB_CORRECTION" "0;0;180"
+			(at 102.87 102.87 0)
+			(effects
