File: sim/sim.kicad_sch (KiCad schematic)
At the start: 0 parts

Commit message: Routing almost finished
Other:
- added sheet 3V3 Filter (3v3_filter.kicad_sch)
Changed lines of the file:
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@@
+	)
+	(sheet
+		(at 154.94 120.65)
+		(size 17.78 11.43)
+		(fields_autoplaced yes)
+		(stroke
+			(width 0.1524)
+			(type solid)
+		)
+		(fill
+			(color 0 0 0 0.0000)
+		)
+		(property "Sheetname" "3V3 Filter"
+			(at 154.94 119.9384 0)
+			(effects
+				(font
+					(size 1.27 1.27)
+				)
+				(justify left bottom)
+			)
+		)
+		(property "Sheetfile" "3v3_filter.kicad_sch"
+			(at 154.94 132.6646 0)
+			(effects
+				(font
+					(size 1.27 1.27)
+				)
+				(justify left top)
+			)
+		)
+		(instances
+			(project "sim"
+				(path "/8bde1ad1-07df-47e7-8106-4608756be5c6"
+					(page "5")
+				)
+			)
+		)
 	)
 	(sheet
